File: prototype/V1.0/board/VFODial/VFODial.sch (KiCad schematic (older format))
At the start: 9 parts

Commit message: Adding pcb data
Parts:
- added C101, C106, C107, C108, C109, C110, C111, C112, C113, C114, C119: 100nF, SM0603, symbol passives:CAP_0603
- added C104, C105: 4.7uF, SM0805, symbol passives:CAP_0805
- added C115, C116, C117, C118: 10uF, SM1206, symbol passives:CAP_1206
- added D101, D102, D103, D104, D105, D106, D107, D108, D109, D110, D111, D112: BAT43W, General_SMD:SOD-123, symbol passives:DIODE
- added J102: SWD Con, Connector_PinHeader_1.27mm:PinHeader_2x05_P1.27mm_Vertical, symbol Connector_Generic:Conn_02x05_Odd_Even
- added J103, J104: Conn_01x04, Connector_PinHeader_2.54mm:PinHeader_1x04_P2.54mm_Vertical, symbol Connector_Generic:Conn_01x04
- added J105: Conn_01x05, Connector_PinHeader_2.54mm:PinHeader_1x05_P2.54mm_Vertical, symbol Connector_Generic:Conn_01x05
- added L101: LED_RGB, Cree:CLMVC-FKA_RGBLED, symbol passives:LED_RGB
- added Q101, Q102, Q103, Q104, Q105, Q106, Q107: BSS138, SOT:SOT-23, symbol NMOS:BSS138
- added R105, R106, R107, R111, R112, R113, R114, R115, R116, R117, R118, R119, R121, R122, R123, R124, R125, R126: 220, SM0603, symbol passives:RES_0603
- added R108, R109, R110: 10, SM0603, symbol passives:RES_0603
- added R120, R127, R129: 10k, SM0603, symbol passives:RES_0603
- added R128: 33.2k, SM0603, symbol passives:RES_0603
- added S101, S102, S103, S104, S105, S106, S107, S108, S109, S110, S111, S112, S113, S114, S115: MX1A-x1-xW, Cherry:MX1A-x1-xW, symbol Cherry_MX:MX1A-x1-xW
- added U102: 3.3uH, Wurth:WE-LHMI_SMD_9.2x8.5x3, symbol passives:IND_SMALL
- added U103: TPS563208_SOT236, SOT:TPS_SOT23-6, symbol tps563208_sot236:TPS563208_SOT236
- J101: renamed from J?; footprint (none) -> Connector_USB:USB_Micro-B_Wuerth_629105150521_CircularHoles; SKU (none) -> 710-629105150521; Vendor (none) -> MOUSER
- U101: renamed from U?; footprint (none) -> Package_QFP:TQFP-48_7x7mm_P0.5mm
- X101: renamed from X?; footprint (none) -> Xtal_SMD:xtal_3.2x2.5; SKU (none) -> 710-830108207109; Vendor (none) -> MOUSER
- gave numbers to parts that had none: 6
Connections:
- net +3V3: now also U101.18 (ADVREFP), U101.19 (AVDD), U101.29 (VDDIO), U101.40 (VDDIO), U101.45 (VDDIO), U101.8 (VDDin), C101.2, C104.1, C105.1, C106.1, C107.1, C108.1, C109.1, C110.1, C114.1, C115.1, C116.1, J102.1 (Pin_1), J104.3 (Pin_3), J105.1 (Pin_1), L101.1 (CA), R111.2, R112.2, R113.2, R114.2, R115.2, R116.2, R117.2, R118.2, R119.2, R121.2, R122.2, R123.2, R124.2, R125.2, R126.2, R128.1, U102.1
- net +5V: now also C117.1, C118.1, J103.1 (Pin_1), U103.3 (VIN), U103.5 (EN)
- net COARSE_COD_N: now also J105.3 (Pin_3)
- net COARSE_COD_P: now also J105.4 (Pin_4)
- net GND: now also C101.1, C104.2, C105.2, C106.2, C107.2, C108.2, C109.2, C110.2, C111.1, C112.1, C113.1, C114.2, C115.2, C116.2, C117.2, C118.2, J102.3 (Pin_3), J102.5 (Pin_5), J102.9 (Pin_9), J103.4 (Pin_4), J104.4 (Pin_4), J105.5 (Pin_5), Q101.2 (S), Q102.2 (S), Q103.2 (S), Q104.2 (S), Q105.2 (S), Q106.2 (S), Q107.2 (S), R120.1, R127.2, R129.1, S113.2, S114.2, S115.2, U103.1 (GND)
- net LCD_CK: now also U101.42 (PA22), J104.2 (Pin_2); no longer U101.44 (PA24)
- net LCD_DA: now also U101.41 (PA21), J104.1 (Pin_1); no longer U101.43 (PA23)
- net SMOOTH_COD_N: now also J103.2 (Pin_2)
- net SMOOTH_COD_P: now also J103.3 (Pin_3)
- net SWDCLK: now also J102.4 (Pin_4)
- net SWDIO: now also J102.2 (Pin_2)
- net ~RESET: now also J102.10 (Pin_10)
- net ROW_0: now reaches U101.20 (PA08)
- net ROW_0: now also S101.1, S104.1, S107.1, S110.1
- net ROW_1: now reaches U101.21 (PA09)
- net ROW_1: now also S102.1, S105.1, S108.1, S111.1
- net COL_1: now reaches U101.22 (PA10)
- net COL_1: now also D104.K, D105.K, D106.K
- net COL_0: now reaches U101.23 (PA11)
- net COL_0: now also D101.K, D102.K, D103.K
- net ROW_2: now reaches U101.24 (PA12)
- net ROW_2: now also S103.1, S106.1, S109.1, S112.1
- net COL_2: now reaches U101.25 (PA27)
- net COL_2: now also D107.K, D108.K, D109.K
- net COL_3: now reaches U101.26 (PA28)
- net COL_3: now also D110.K, D111.K, D112.K
- net MAIN2_LEDS: now reaches U101.27 (PA29)
- net MAIN2_LEDS: now also Q106.1 (G), Q107.1 (G), R129.2
- net MAIN_LEDS: now reaches U101.3 (PA02)
- net MAIN_LEDS: now also Q101.1 (G), Q104.1 (G), R120.2
- net at U101.30 (PA30): now also R107.2
- net at U101.31 (PA31): now also R106.2
- net at U101.32 (PA13): now also R105.2
- net PB1_LED: now reaches U101.33 (PA14)
- net PB1_LED: now also Q105.1 (G)
- net PB2_LED: now reaches U101.34 (PA15)
- net PB2_LED: now also Q103.1 (G)
- net PB3_LED: now reaches U101.35 (PA16)
- net PB3_LED: now also Q102.1 (G)
- net PB1: now reaches U101.36 (PA17)
- net PB1: now also C111.2, R108.2
- net PB2: now reaches U101.37 (PA18)
- net PB2: now also C112.2, R109.2
- net PB3: now reaches U101.38 (PA19)
- net PB3: now also C113.2, R110.2
- net ROT_PB: now reaches U101.39 (PA20)
- net ROT_PB: now also J105.2 (Pin_2)
- net at U101.5 (VDDCore): now also U101.7 (VDDout)
- new net: D101.A, S101.2
- new net: R111.1, S101.3
- new net: Q101.3 (D), S101.4, S102.4, S103.4
- new net: D102.A, S102.2
- new net: R112.1, S102.3
- new net: D103.A, S103.2
- new net: R113.1, S103.3
- new net: D104.A, S104.2
- new net: R117.1, S104.3
- new net: Q104.3 (D), S104.4, S105.4, S106.4
- new net: D105.A, S105.2
- new net: R118.1, S105.3
- new net: D106.A, S106.2
- new net: R119.1, S106.3
- new net: D107.A, S107.2
- new net: R121.1, S107.3
- new net: Q106.3 (D), S107.4, S108.4, S109.4
- new net: D108.A, S108.2
- new net: R122.1, S108.3
- new net: D109.A, S109.2
- new net: R123.1, S109.3
- new net: D110.A, S110.2
- new net: R124.1, S110.3
- new net: Q107.3 (D), S110.4, S111.4, S112.4
- new net: D111.A, S111.2
- new net: R125.1, S111.3
- new net: D112.A, S112.2
- new net: R126.1, S112.3
- new net: L101.2 (BK), R107.1
- new net: L101.3 (GK), R106.1
- new net: L101.4 (RK), R105.1
- new net: R108.1, S113.1
- new net: R114.1, S113.3
- new net: Q105.3 (D), S113.4
- new net: R109.1, S114.1
- new net: R115.1, S114.3
- new net: Q103.3 (D), S114.4
- new net: R110.1, S115.1
- new net: R116.1, S115.3
- new net: Q102.3 (D), S115.4
- new net: R127.1, R128.2, U103.4 (VFB)
- new net: C119.2, U103.6 (VBST)
- new net SWO: J102.6 (Pin_6), U101.43 (PA23)
- new net psw: C119.1, U102.2, U103.2 (SW)
- no-connect marks 3 -> 6
Other:
- note added: "Also put the internal regulator in LDO mode."
